File: Hardware/ArduSynth.sch (KiCad schematic (older format))
At the start: 21 parts, among them J1 STEREO_JACK_3.5MM, J2 STEREO_JACK_3.5MM, P1 ARD_CONN_8, P2 ADR_CONN_6, P3 ARD_CONN_10, P4 ARD_CONN_8, SW1 SW_12X12MM

Commit message: Fixed lables on sch
Connections:
- net labels removed: VCF_PEAK
Changed lines of the file:
@@
 LIBS:Capacitor_0p01uf
 LIBS:Capacitor_0p1uf
+LIBS:sw_12x12mm
 LIBS:ArduSynth-cache
 EELAYER 27 0
@@
 Sheet 1 1
 Title "ArduSynth Shield"
-Date "27 nov 2014"
+Date "1 dec 2014"
 Rev "A"
 Comp "Electronics Is Fun / uCHobby"
@@
 Text Label 4750 3750 0    60   ~ 0
 GND
-Text Label 5500 6900 0    60   ~ 0
-VCF_PEAK
 Text Label 5600 6800 0    60   ~ 0
 ADJ2
-Text Label 6400 6650 0    60   ~ 0
+Text Label 6400 6700 0    60   ~ 0
 ADJ3
-Text Label 7200 6600 0    60   ~ 0
-ADJ4
-Text Label 8150 6450 0    60   ~ 0
-ADJ5
 Text Label 12000 6700 0    60   ~ 0
 TRIGGER
-Text Label 14900 6250 0    60   ~ 0
+Text Label 14600 6250 0    60   ~ 0
 AUDIO OUT
 Text Label 4900 6900 0    60   ~ 0
 ADJ1
-Text Label 5600 6800 0    60   ~ 0
-ADJ3
 Text Label 7050 6600 0    60   ~ 0
 ADJ4
 Text Label 8200 6500 0    60   ~ 0
 ADJ5
-Text Label 12300 3750 0    60   ~ 0
-ADJ3
-Text Label 12500 6850 0    60   ~ 0
-ADJ3
 Text Label 12450 8000 0    60   ~ 0
 GND

Commit message: Updated symbols for Arduino and placement
Parts:
- removed P1, P4: ARD_CONN_8, ~, symbol ARD_CONN_8
- removed P2: ADR_CONN_6, ~, symbol ADR_CONN_6
- removed P3: ARD_CONN_10, ~, symbol ARD_CONN_10
- added U1: ARDUINOR3, ArduinoR3, symbol ARDUINOR3
- C1, C2, C3: footprint ~ -> C1
- D1: footprint ~ -> LED-3MM
- R1, R2, R3, R4: footprint ~ -> R4
- RV1, RV2, RV3, RV4, RV5, RV6: footprint ALPS-10x10mm -> POT_CMS
- SW1: footprint TH_12x12MM -> SW_PUSH_SMALL
Other:
- note removed: "(PWM Pins D3, D5, D6, D9, D10, D11)"
- note removed: "3.3V"
- note removed: "5V"
- note removed: "A0"
- note removed: "A1\n"
- note removed: "A2\n"
- note removed: "A3\n"
- note removed: "A4"
- note removed: "A5"
- note removed: "ARDUINO HEADERS"
- note removed: "AREF"
- note removed: "D10-"
- note removed: "D11-"
- note removed: "D12"
- note removed: "D13"
- note removed: "D2\n"
- note removed: "D3-\n"
- note removed: "D4"
- note removed: "D5-"
- note removed: "D6-"
- note removed: "D7"
- note removed: "D8"
- note removed: "D9-"
- note removed: "GND"
- note removed: "IOREF"
- note removed: "NC"
- note removed: "RESET"
- note removed: "RX<-0"
- note removed: "SCL"
- note removed: "SDA"
- note removed: "TX->1"
- note removed: "Vin"
- moved on the sheet: D1, J1, J2, R1, R2, R3, R4, RV1, RV2, RV3, RV4, RV5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
